File: stm8l151.kicad_pcb (KiCad board)
At the start: 2 copper layers, 38.1 x 50 mm, 43 parts, among them J1 PWR_MCU, J10 C, J11 SWIM, J12 I²C, J13 pwr, J14 pwr, J15 pwr, J2 PWR_EEP, J5 C, J6 C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

Commit message: Add files via upload
Parts:
- moved G*** 0.90 mm to (38.1, 42.4)
- moved Y2 0.25 mm to (43.9, 36.3)
Routing:
- net /A4: track 20.7 -> 21.6 mm
Other:
- board text added: "KBS 2022"
