File: stm8l151.kicad_sch (KiCad schematic)
At the start: 41 parts, among them J1 PWR_MCU, J10 C, J11 SWIM, J12 I²C, J13 pwr, J14 pwr, J15 pwr, J2 PWR_EEP, J5 C, J6 C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

Commit message: Add files via upload
Other:
- note added: "100uA"
- moved on the sheet: C1, C2, C3, D1, J1, J13, J14, J15, J2, U1
